Commit message: feat: Add Camera Sensor in URDF Robot

File: src/caramelo_description/urdf/bumperbot.urdf.xacro (robot description, xacro)
@@ -1,4 +1,4 @@
 <?xml version="1.0"?>
-<robot name="bumperbot" xmlns:xacro="http://ros.org/wiki/xacro">
+<robot name="caramelo" xmlns:xacro="http://ros.org/wiki/xacro">
   <!-- Start GZ or Ignition depending on ROS 2 Version -->
   <xacro:arg name="is_ignition" default="true"/>
@@ -9,4 +9,7 @@
   <!-- Include ros2_control Plugins -->
   <xacro:include filename="$(find caramelo_description)/urdf/bumperbot_ros2_control.xacro" />
+  <!-- ==================== -->
+  <!--       BASE LINK      -->
+  <!-- ==================== -->
   <link name="base_footprint"/>
   <link name="base_link">
@@ -37,4 +40,7 @@
     <origin xyz="0 0 0.033" rpy="0 0 0"/>
   </joint>
+  <!-- ==================== -->
+  <!--   WHEEL RIGHT LINK   -->
+  <!-- ==================== -->
   <link name="wheel_right_link">
     <inertial>
@@ -65,4 +71,7 @@
     <axis xyz="0 1 0" />
   </joint>
+  <!-- ==================== -->
+  <!--   WHEEL LEFT LINK    -->
+  <!-- ==================== -->
   <link
     name="wheel_left_link">
@@ -94,4 +103,7 @@
     <axis xyz="0 1 0" />
   </joint>
+  <!-- ==================== -->
+  <!--   CASTER FRONT LINK   -->
+  <!-- ==================== -->
   <link name="caster_front_link">
     <inertial>
@@ -122,4 +134,7 @@
     <axis xyz="0 0 0" />
   </joint>
+  <!-- ==================== -->
+  <!--   CASTER REAR LINK   -->
+  <!-- ==================== -->
   <link name="caster_rear_link">
     <inertial>
@@ -150,4 +165,7 @@
     <axis xyz="0 0 0" />
   </joint>
+  <!-- ==================== -->
+  <!--   IMU LINK          -->
+  <!-- ==================== -->
   <link name="imu_link">
     <inertial>
@@ -178,4 +196,7 @@
     <axis xyz="0 0 0" />
   </joint>
+  <!-- ==================== -->
+  <!--   LASER LINK        -->
+  <!-- ==================== -->
   <link name="laser_link">
     <inertial>
@@ -206,4 +227,42 @@
     <axis xyz="0 0 0" />
   </joint>
+  <!-- ==================== -->
+  <!--   CAMERA LINK       -->
+  <!-- ==================== -->
+  <link name="camera_link">
+    <visual>
+      <geometry>
+        <box size="0.03 0.06 0.03"/>
+      </geometry>
+      <material name="camera_dark">
+        <color rgba="0.05 0.05 0.05 1.0"/>
+      </material>
+    </visual>
+    <collision>
+      <geometry>
+        <box size="0.03 0.06 0.03"/>
+      </geometry>
+    </collision>
+    <inertial>
+      <mass value="0.05"/>
+      <inertia ixx="0.00005" ixy="0" ixz="0"
+               iyy="0.00005" iyz="0" izz="0.00005"/>
+    </inertial>
+  </link>
+  <joint name="camera_joint" type="fixed">
+    <parent link="base_link" />
+    <child link="camera_link" />
+    <origin xyz="0.08 0 0.04" rpy="0 0 0" />
+  </joint>
+  <link name="camera_link_optical"/>
+  <!-- Optical frame: ROS convention (x-right, y-down, z-forward) -->
+  <joint name="camera_optical_joint" type="fixed">
+    <parent link="camera_link"/>
+    <child link="camera_link_optical"/>
+    <origin xyz="0 0 0" rpy="-1.5708 0 -1.5708"/>
+  </joint>
+  <!-- ==================== -->
+  <!--   MATERIALS         -->
+  <!-- ==================== -->
   <material name="blue">
     <color rgba="0 0 1 1"/>

File: src/caramelo_description/urdf/bumperbot_gazebo.xacro (robot description, xacro)
@@ -1,4 +1,7 @@
 <?xml version="1.0"?>
-<robot name="bumperbot" xmlns:xacro="http://ros.org/wiki/xacro">
+<robot name="caramelo" xmlns:xacro="http://ros.org/wiki/xacro">
+  <!-- ==================== -->
+  <!--    GAZEBO PLUGINS    -->
+  <!-- ==================== -->
   <!-- Wheels -->
   <gazebo reference="wheel_left_link">
@@ -143,3 +146,31 @@
     </sensor>
   </gazebo>
+  <!-- Camera Sensor -->
+  <gazebo reference="camera_link">
+    <sensor name="camera" type="camera">
+      <pose>0 0 0 0 0 0</pose>
+      <topic>camera/image</topic>
+      <gz_frame_id>camera_link_optical</gz_frame_id>
+      <update_rate>30</update_rate>
+      <always_on>true</always_on>
+      <visualize>true</visualize>
+      <camera>
+        <horizontal_fov>1.3962634</horizontal_fov>
+        <image>
+          <width>640</width>
+          <height>480</height>
+          <format>R8G8B8</format>
+        </image>
+        <clip>
+          <near>0.05</near>
+          <far>50.0</far>
+        </clip>
+        <noise>
+          <type>gaussian</type>
+          <mean>0.0</mean>
+          <stddev>0.005</stddev>
+        </noise>
+      </camera>
+    </sensor>
+  </gazebo>
 </robot>

File: src/caramelo_description/urdf/bumperbot_ros2_control.xacro (robot description, xacro)
@@ -1,4 +1,4 @@
 <?xml version="1.0"?>
-<robot xmlns:xacro="http://www.ros.org/wiki/xacro" name="bumperbot">
+<robot xmlns:xacro="http://www.ros.org/wiki/xacro" name="caramelo">
     <ros2_control name="RobotSystem" type="system">
         <!-- ros2_control Gazebo -->
